File: core/imx233-core.sch (KiCad schematic (older format))
At the start: 57 parts, among them J1 Conn_01x15, J2 Conn_01x19, J3 Conn_01x19, J4 Conn_01x02, J5 USB_B_Micro, U1 MCIMX233CAG4C, U2 MT46V32M16, X1 24MHz

Commit message: core: Add ESD protection to USB
Update mx233 symbol & footprint library.
Parts:
- removed TF1: TF_Card, Lib:XKXFS-N02-XXT, symbol LIB:TF_Card
- removed U1: MCIMX233CAG4C, Lib:LQFP-128_14x14_Pitch0.4mm, symbol LIB:MCIMX233CAG4C
- removed U2: MT46V32M16, Lib:TSSOP-66_400mil_P0.65mm, symbol LIB:MT46V32M16
- removed X1: 24MHz, Lib:Crystal_SMD_3225-4P_3.2x2.5mm, symbol LIB:XTAL-4
- added TF1: TF_Card, Library:XKXFS-N02-XXT, symbol Library:TF_Card
- added U1: MCIMX233CAG4C, Library:LQFP-128_14x14_Pitch0.4mm, symbol Library:MCIMX233CAG4C
- added U2: MT46V32M16, Library:TSSOP-66_400mil_P0.65mm, symbol Library:MT46V32M16
- added U3: SR05, Package_TO_SOT_SMD:SOT-143, symbol Library:SR05
- added X1: 24MHz, Library:Crystal_SMD_3225-4P_3.2x2.5mm, symbol Library:XTAL-4
- J5: footprint Lib:USB_Micro-Molex -> Library:USB_Micro-Molex
- L1: footprint Lib:Inductor-4x4 -> Library:Inductor-4x4
Connections:
- wire segments 449 -> 453
Changed lines of the file:
@@
 F 0 "L1" V 7450 4850 50  0000 C CNN
 F 1 "22uH" V 7350 5000 50  0000 C CNN
-F 2 "Lib:Inductor-4x4" H 7400 5000 50  0001 C CNN
+F 2 "Library:Inductor-4x4" H 7400 5000 50  0001 C CNN
 F 3 "~" H 7400 5000 50  0001 C CNN
 	1    7400 5000
@@
 	1650 5500 2100 5500
 Wire Wire Line
-	10050 10100 10500 10100
-Wire Wire Line
-	10050 10000 10500 10000
-Wire Wire Line
 	1650 7100 2100 7100
 Wire Wire Line
@@
 Text Label 2100 2350 2    50   ~ 0
 SSP_CMD
-$Comp
-L LIB:MCIMX233CAG4C U1
-U 1 1 5DC52A97
-P 5550 5300
-F 0 "U1" H 5450 8887 60  0000 C CNN
-F 1 "MCIMX233CAG4C" H 5450 8781 60  0000 C CNN
-F 2 "Lib:LQFP-128_14x14_Pitch0.4mm" H 4250 6100 60  0001 C CNN
-F 3 "" H 4250 6100 60  0001 C CNN
-	1    5550 5300
-	1    0    0    -1
-$EndComp
-$Comp
-L LIB:MT46V32M16 U2
-U 1 1 5DC60DEE
-P 12450 7100
-F 0 "U2" H 12450 9487 60  0000 C CNN
-F 1 "MT46V32M16" H 12450 9381 60  0000 C CNN
-F 2 "Lib:TSSOP-66_400mil_P0.65mm" H 13350 7500 60  0001 C CNN
-F 3 "" H 13350 7500 60  0001 C CNN
-	1    12450 7100
-	1    0    0    -1
-$EndComp
-$Comp
-L LIB:XTAL-4 X1
-U 1 1 5DCB7A83
-P 9000 2750
-F 0 "X1" H 9025 3087 60  0000 C CNN
-F 1 "24MHz" H 9025 2981 60  0000 C CNN
-F 2 "Lib:Crystal_SMD_3225-4P_3.2x2.5mm" H 9400 2500 60  0001 C CNN
-F 3 "" H 9400 2500 60  0001 C CNN
-	1    9000 2750
-	1    0    0    -1
-$EndComp
 Wire Wire Line
 	6750 2700 8250 2700
@@
 Wire Wire Line
 	9000 3100 8450 3100
-$Comp
-L LIB:TF_Card TF1
-U 1 1 5E12ABC0
-P 6950 9900
-F 0 "TF1" H 7050 10487 60  0000 C CNN
-F 1 "TF_Card" H 7050 10381 60  0000 C CNN
-F 2 "Lib:XKXFS-N02-XXT" H 6250 10400 60  0001 C CNN
-F 3 "" H 6250 10400 60  0001 C CNN
-	1    6950 9900
-	1    0    0    -1
-$EndComp
 Wire Wire Line
 	1650 3450 1750 3450
@@
 F 0 "J5" H 10570 9989 50  0000 R CNN
 F 1 "USB_B_Micro" H 10570 9898 50  0000 R CNN
-F 2 "Lib:USB_Micro-Molex" H 10950 9950 50  0001 C CNN
+F 2 "Library:USB_Micro-Molex" H 10950 9950 50  0001 C CNN
 F 3 "~" H 10950 9950 50  0001 C CNN
 	1    10800 10000
@@
 Text Label 2100 4500 2    50   ~ 0
 P0_17
+Wire Wire Line
+	9300 10000 9200 10000
+$Comp
+L power:+5V #PWR07
+U 1 1 5F4C9C73
+P 9200 9900
+F 0 "#PWR07" H 9200 9750 50  0001 C CNN
+F 1 "+5V" H 9100 10050 50  0000 L CNN
+F 2 "" H 9200 9900 50  0001 C CNN
+F 3 "" H 9200 9900 50  0001 C CNN
+	1    9200 9900
+	1    0    0    -1
+$EndComp
+Wire Wire Line
+	9200 9900 9200 10000
+$Comp
+L power:GND #PWR08
+U 1 1 5F515A0B
+P 9200 10200
+F 0 "#PWR08" H 9200 9950 50  0001 C CNN
+F 1 "GND" H 9205 10027 50  0000 C CNN
+F 2 "" H 9200 10200 50  0001 C CNN
+F 3 "" H 9200 10200 50  0001 C CNN
+	1    9200 10200
+	1    0    0    -1
+$EndComp
+Wire Wire Line
+	9200 10200 9200 10100
+Wire Wire Line
+	9200 10100 9300 10100
+Wire Wire Line
+	9950 10000 10500 10000
+Wire Wire Line
+	9950 10100 10500 10100
+$Comp
+L Library:MCIMX233CAG4C U1
+U 1 1 5F515ABD
+P 5550 5300
+F 0 "U1" H 5450 8887 60  0000 C CNN
+F 1 "MCIMX233CAG4C" H 5450 8781 60  0000 C CNN
+F 2 "Library:LQFP-128_14x14_Pitch0.4mm" H 4250 6100 60  0001 C CNN
+F 3 "" H 4250 6100 60  0001 C CNN
+	1    5550 5300
+	1    0    0    -1
+$EndComp
+$Comp
+L Library:TF_Card TF1
+U 1 1 5F51A132
+P 6950 9900
+F 0 "TF1" H 7050 10487 60  0000 C CNN
+F 1 "TF_Card" H 7050 10381 60  0000 C CNN
+F 2 "Library:XKXFS-N02-XXT" H 6250 10400 60  0001 C CNN
+F 3 "" H 6250 10400 60  0001 C CNN
+	1    6950 9900
+	1    0    0    -1
+$EndComp
+$Comp
+L Library:MT46V32M16 U2
+U 1 1 5F51D448
+P 12450 7100
+F 0 "U2" H 12450 9487 60  0000 C CNN
+F 1 "MT46V32M16" H 12450 9381 60  0000 C CNN
+F 2 "Library:TSSOP-66_400mil_P0.65mm" H 13350 7500 60  0001 C CNN
+F 3 "" H 13350 7500 60  0001 C CNN
+	1    12450 7100
+	1    0    0    -1
+$EndComp
+$Comp
+L Library:SR05 U3
+U 1 1 5F51FD97
+P 9650 10050
+F 0 "U3" H 9625 10365 50  0000 C CNN
+F 1 "SR05" H 9625 10274 50  0000 C CNN
+F 2 "Package_TO_SOT_SMD:SOT-143" H 9650 10000 50  0001 C CNN
+F 3 "" H 9650 10000 50  0001 C CNN
+	1    9650 10050
+	1    0    0    -1
+$EndComp
+$Comp
+L Library:XTAL-4 X1
+U 1 1 5F52187B
+P 9000 2750
+F 0 "X1" H 9025 3087 60  0000 C CNN
+F 1 "24MHz" H 9025 2981 60  0000 C CNN
+F 2 "Library:Crystal_SMD_3225-4P_3.2x2.5mm" H 9400 2500 60  0001 C CNN
+F 3 "" H 9400 2500 60  0001 C CNN
+	1    9000 2750
+	1    0    0    -1
+$EndComp
 $EndSCHEMATC
